Commit message: fix mass value from 0.0.0 to 0.0

File: resources/robots/XBot/urdf/XBot-L.urdf (robot description, URDF)
Before this commit: robot XBot-L, 91 links, 90 joints
Links:
- link left_hand_ee_link: mass 0.0.0 -> 0.0
- link left_hand_index_rota_link2: mass 0.0.0 -> 0.0
- link left_hand_index_tip: mass 0.0.0 -> 0.0
- link left_hand_link: mass 0.0.0 -> 0.0
- link left_hand_mid_link1: mass 0.0.0 -> 0.0
- link left_hand_mid_link2: mass 0.0.0 -> 0.0
- link left_hand_mid_tip: mass 0.0.0 -> 0.0
- link left_hand_pinky_link1: mass 0.0.0 -> 0.0
- link left_hand_pinky_link2: mass 0.0.0 -> 0.0
- link left_hand_pinky_tip: mass 0.0.0 -> 0.0
- link left_hand_ring_link1: mass 0.0.0 -> 0.0
- link left_hand_ring_link2: mass 0.0.0 -> 0.0
- link left_hand_ring_tip: mass 0.0.0 -> 0.0
- link left_hand_thumb_bend_link: mass 0.0.0 -> 0.0
- link left_hand_thumb_rota_link1: mass 0.0.0 -> 0.0
- link left_hand_thumb_rota_link2: mass 0.0.0 -> 0.0
- link left_hand_thumb_tip: mass 0.0.0 -> 0.0
- link right_hand_ee_link: mass 0.0.0 -> 0.0
- link right_hand_index_rota_link2: mass 0.0.0 -> 0.0
- link right_hand_index_tip: mass 0.0.0 -> 0.0
- link right_hand_link: mass 0.0.0 -> 0.0
- link right_hand_mid_link1: mass 0.0.0 -> 0.0
- link right_hand_mid_link2: mass 0.0.0 -> 0.0
- link right_hand_mid_tip: mass 0.0.0 -> 0.0
- link right_hand_pinky_link1: mass 0.0.0 -> 0.0
- link right_hand_pinky_link2: mass 0.0.0 -> 0.0
- link right_hand_pinky_tip: mass 0.0.0 -> 0.0
- link right_hand_ring_link1: mass 0.0.0 -> 0.0
- link right_hand_ring_link2: mass 0.0.0 -> 0.0
- link right_hand_ring_tip: mass 0.0.0 -> 0.0
- link right_hand_thumb_bend_link: mass 0.0.0 -> 0.0
- link right_hand_thumb_rota_link1: mass 0.0.0 -> 0.0
- link right_hand_thumb_rota_link2: mass 0.0.0 -> 0.0
- link right_hand_thumb_rota_tip: mass 0.0.0 -> 0.0

Commit message: yjhbot

File: resources/robots/XBot/urdf/XBot-L.urdf (robot description, URDF)
Before this commit: robot XBot-L, 91 links, 90 joints
Joints:
- joint left_elbow_pitch_joint: type fixed -> revolute
- joint left_shoulder_pitch_joint: type fixed -> revolute
- joint left_wrist_roll_joint: type fixed -> revolute
- joint right_elbow_pitch_joint: type fixed -> revolute
- joint right_shoulder_pitch_joint: type fixed -> revolute
- joint right_wrist_roll_joint: type fixed -> revolute
